File: projects/DEC/Mxxx/M705/M705D.sch (EAGLE design)
At the start: 48 parts

Commit message: Remove vestigial use of library dec-r.  Henceforth, dec-m is the library for dec modules.
Connections:
- removed net NC: E11A.CLR, E11A.PRE, E11B.CLR, E11B.PRE, E1A.PRE, E1B.PRE, E2A.PRE, E2B.PRE, E3A.PRE, E3B.PRE, E4A.PRE, E4B.PRE, E5A.PRE
Changed lines of the file:
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@@
 <part name="V3" library="supply2" deviceset="GND" device=""/>
 <part name="V7" library="supply2" deviceset="GND" device=""/>
-<part name="U$1" library="dec-r" deviceset="NC" device=""/>
-<part name="U$4" library="dec-r" deviceset="NC" device=""/>
-<part name="U$7" library="dec-r" deviceset="NC" device=""/>
-<part name="U$8" library="dec-r" deviceset="NC" device=""/>
-<part name="U$9" library="dec-r" deviceset="NC" device=""/>
-<part name="U$10" library="dec-r" deviceset="NC" device=""/>
-<part name="U$11" library="dec-r" deviceset="NC" device=""/>
-<part name="U$12" library="dec-r" deviceset="NC" device=""/>
-<part name="U$13" library="dec-r" deviceset="NC" device=""/>
-<part name="U$14" library="dec-r" deviceset="NC" device=""/>
-<part name="U$15" library="dec-r" deviceset="NC" device=""/>
-<part name="U$16" library="dec-r" deviceset="NC" device=""/>
-<part name="U$17" library="dec-r" deviceset="NC" device=""/>
 </parts>
 <sheets>
@@
 <instance part="V3" gate="GND" x="116.84" y="241.3"/>
 <instance part="V7" gate="GND" x="304.8" y="71.12"/>
-<instance part="U$1" gate="NC" x="304.8" y="238.76" rot="MR180"/>
-<instance part="U$4" gate="NC" x="304.8" y="218.44" rot="MR180"/>
-<instance part="U$7" gate="NC" x="304.8" y="198.12" rot="MR180"/>
-<instance part="U$8" gate="NC" x="304.8" y="177.8" rot="MR180"/>
-<instance part="U$9" gate="NC" x="304.8" y="157.48" rot="MR180"/>
-<instance part="U$10" gate="NC" x="304.8" y="137.16" rot="MR180"/>
-<instance part="U$11" gate="NC" x="304.8" y="116.84" rot="MR180"/>
-<instance part="U$12" gate="NC" x="304.8" y="96.52" rot="MR180"/>
-<instance part="U$13" gate="NC" x="304.8" y="55.88" rot="MR180"/>
-<instance part="U$14" gate="NC" x="215.9" y="50.8" rot="MR180"/>
-<instance part="U$15" gate="NC" x="215.9" y="60.96" rot="MR180"/>
-<instance part="U$16" gate="NC" x="215.9" y="88.9" rot="MR180"/>
-<instance part="U$17" gate="NC" x="215.9" y="99.06" rot="MR180"/>
 </instances>
 <busses>
@@
 </segment>
 </net>
-<net name="NC" class="0">
-<segment>
-<pinref part="E1" gate="A" pin="PRE"/>
-<pinref part="U$1" gate="NC" pin="NC"/>
-</segment>
-<segment>
-<pinref part="E1" gate="B" pin="PRE"/>
-<pinref part="U$4" gate="NC" pin="NC"/>
-</segment>
-<segment>
-<pinref part="E2" gate="A" pin="PRE"/>
-<pinref part="U$7" gate="NC" pin="NC"/>
-</segment>
-<segment>
-<pinref part="E2" gate="B" pin="PRE"/>
-<pinref part="U$8" gate="NC" pin="NC"/>
-</segment>
-<segment>
-<pinref part="E3" gate="A" pin="PRE"/>
-<pinref part="U$9" gate="NC" pin="NC"/>
-</segment>
-<segment>
-<pinref part="E3" gate="B" pin="PRE"/>
-<pinref part="U$10" gate="NC" pin="NC"/>
-</segment>
-<segment>
-<pinref part="E4" gate="A" pin="PRE"/>
-<pinref part="U$11" gate="NC" pin="NC"/>
-</segment>
-<segment>
-<pinref part="E4" gate="B" pin="PRE"/>
-<pinref part="U$12" gate="NC" pin="NC"/>
-</segment>
-<segment>
-<pinref part="E5" gate="A" pin="PRE"/>
-<pinref part="U$13" gate="NC" pin="NC"/>
-</segment>
-<segment>
-<pinref part="E11" gate="B" pin="CLR"/>
-<pinref part="U$14" gate="NC" pin="NC"/>
-</segment>
-<segment>
-<pinref part="E11" gate="B" pin="PRE"/>
-<pinref part="U$15" gate="NC" pin="NC"/>
-</segment>
-<segment>
-<pinref part="E11" gate="A" pin="CLR"/>
-<pinref part="U$16" gate="NC" pin="NC"/>
-</segment>
-<segment>
-<pinref part="E11" gate="A" pin="PRE"/>
-<pinref part="U$17" gate="NC" pin="NC"/>
-</segment>
-</net>
 </nets>
 </sheet>
 </sheets>
+<errors>
+</errors>
 </schematic>
 </drawing>
