File: projects/RX08/kludge.brd (EAGLE design)
At the start: 160 x 100 mm, 10 parts

Commit message: Where possible, map 74xx-jameco to 74xx-us. Moved the 7438 to dec-con.lbr. Also changed the spelling of CRYTAL to CRYSTAL.
Parts:
- E17: value 74LS76N -> 7476N; device 74xx-jameco:DIL16 -> 74xx-us:DIL16
Changed lines of the file:
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@@
 <element name="P19" library="ic-package" package="DIL16" value="" x="34.29" y="52.07" rot="R180"/>
 <element name="P17" library="ic-package" package="DIL16" value="" x="59.69" y="52.07" rot="R180"/>
-<element name="E17" library="74xx-jameco" package="DIL16" value="74LS76N" x="59.69" y="67.31" rot="R180"/>
+<element name="E17" library="74xx-us" package="DIL16" value="7476N" x="59.69" y="67.31" rot="R180"/>
 <element name="SV1" library="con-lsta" package="FE07" value="" x="60.96" y="78.74" rot="R180">
 <attribute name="OC_NEWARK" value="unknown" x="60.96" y="78.74" size="1.778" layer="27" rot="R180" display="off"/>
