File: projects/FlipChip/InnerConnector.sch (EAGLE design)
At the start: 4 parts

Commit message: Replace all instances of the JP2Q jumper with one from dec-con, as the JUMPER library has pins 2 and 3 swapped.
Parts:
- P1, P2: device jumper:JP2Q -> dec-con:JP2Q
Changed lines of the file:
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@@
 <part name="U$1" library="dec-con" deviceset="EDGE-2" device="CONNECTOR"/>
 <part name="SV1" library="con-lstb" deviceset="MA18-2" device=""/>
-<part name="P2" library="jumper" deviceset="JP2Q" device=""/>
-<part name="P1" library="jumper" deviceset="JP2Q" device=""/>
+<part name="P2" library="dec-con" deviceset="JP2Q" device=""/>
+<part name="P1" library="dec-con" deviceset="JP2Q" device=""/>
 </parts>
 <sheets>
