File: projects/DEC/Gxxx/G020/G020X.sch (EAGLE design)
At the start: 84 parts, among them Q1 2N3009, Q2 2N3009

Commit message: Walk the project tree, making things pass current design rules.
Changed lines of the file:
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@@
 <pinref part="E2A" gate="A" pin="I0"/>
 <pinref part="U$1" gate="D1" pin="1"/>
+<label x="109.22" y="109.22" size="1.778" layer="95" rot="R90"/>
 </segment>
 </net>
@@
 <pinref part="E2A" gate="D" pin="O"/>
 <pinref part="U$1" gate="C1" pin="1"/>
+<label x="137.16" y="160.02" size="1.778" layer="95" rot="R90"/>
 </segment>
 <segment>
@@
 <pinref part="E2A" gate="A" pin="O"/>
 <pinref part="U$1" gate="S1" pin="1"/>
+<label x="137.16" y="116.84" size="1.778" layer="95" rot="R90"/>
 </segment>
 <segment>
@@
 <pinref part="E2A" gate="B" pin="I1"/>
 <pinref part="U$1" gate="R1" pin="1"/>
+<label x="109.22" y="22.86" size="1.778" layer="95" rot="R90"/>
 </segment>
 </net>
@@
 </sheet>
 </sheets>
+<errors>
+</errors>
 </schematic>
 </drawing>
