File: projects/DEC/Mxxx/M116/M116A.brd (EAGLE design)
At the start: 125.7 x 62.2 mm, 12 parts

Commit message: Walk the project tree, making things pass current design rules.
Changed lines of the file:
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@@
 <param name="mdViaViaSameLayer" value="8mil"/>
 <param name="mnLayersViaInSmd" value="2"/>
-<param name="mdCopperDimension" value="25mil"/>
+<param name="mdCopperDimension" value="13mil"/>
 <param name="mdDrill" value="10mil"/>
 <param name="mdSmdStop" value="0mil"/>
@@
 <wire x1="117.1702" y1="29.5402" x2="117.7925" y2="29.5275" width="0.4064" layer="16"/>
 <wire x1="116.84" y1="29.21" x2="117.1702" y2="29.5402" width="0.4064" layer="16"/>
-<wire x1="111.76" y1="29.21" x2="116.84" y2="29.21" width="0.4064" layer="16"/>
-<wire x1="107.95" y1="25.4" x2="111.76" y2="29.21" width="0.4064" layer="16"/>
-<wire x1="96.52" y1="25.4" x2="107.95" y2="25.4" width="0.4064" layer="16"/>
+<wire x1="110.49" y1="29.21" x2="116.84" y2="29.21" width="0.4064" layer="16"/>
+<wire x1="106.68" y1="25.4" x2="110.49" y2="29.21" width="0.4064" layer="16"/>
+<wire x1="96.52" y1="25.4" x2="106.68" y2="25.4" width="0.4064" layer="16"/>
 <wire x1="93.98" y1="27.94" x2="96.52" y2="25.4" width="0.4064" layer="16"/>
 </signal>
@@
 <wire x1="117.1956" y1="7.2644" x2="117.7925" y2="7.3025" width="0.4064" layer="16"/>
 <wire x1="116.84" y1="7.62" x2="117.1956" y2="7.2644" width="0.4064" layer="16"/>
-<wire x1="111.76" y1="7.62" x2="116.84" y2="7.62" width="0.4064" layer="16"/>
-<wire x1="110.49" y1="8.89" x2="111.76" y2="7.62" width="0.4064" layer="16"/>
-<wire x1="97.79" y1="8.89" x2="110.49" y2="8.89" width="0.4064" layer="16"/>
+<wire x1="110.49" y1="7.62" x2="116.84" y2="7.62" width="0.4064" layer="16"/>
+<wire x1="109.22" y1="8.89" x2="110.49" y2="7.62" width="0.4064" layer="16"/>
+<wire x1="97.79" y1="8.89" x2="109.22" y2="8.89" width="0.4064" layer="16"/>
 <wire x1="96.52" y1="7.62" x2="97.79" y2="8.89" width="0.4064" layer="16"/>
 </signal>
@@
 <wire x1="117.1448" y1="48.5648" x2="117.7925" y2="48.5775" width="0.4064" layer="16"/>
 <wire x1="116.84" y1="48.26" x2="117.1448" y2="48.5648" width="0.4064" layer="16"/>
-<wire x1="111.76" y1="48.26" x2="116.84" y2="48.26" width="0.4064" layer="16"/>
-<wire x1="109.22" y1="45.72" x2="111.76" y2="48.26" width="0.4064" layer="16"/>
-<wire x1="97.79" y1="45.72" x2="109.22" y2="45.72" width="0.4064" layer="16"/>
+<wire x1="110.49" y1="48.26" x2="116.84" y2="48.26" width="0.4064" layer="16"/>
+<wire x1="107.95" y1="45.72" x2="110.49" y2="48.26" width="0.4064" layer="16"/>
+<wire x1="97.79" y1="45.72" x2="107.95" y2="45.72" width="0.4064" layer="16"/>
 <wire x1="96.52" y1="46.99" x2="97.79" y2="45.72" width="0.4064" layer="16"/>
 </signal>
