File: projects/DEC/Mxxx/M220/M220pal.sch (EAGLE design)
At the start: 25 parts

Commit message: Where possible, map 74xx-jameco to 74xx-us. Moved the 7438 to dec-con.lbr. Also changed the spelling of CRYTAL to CRYSTAL.
Parts:
- E3, E4: device 74xx-jameco:74S20N -> 74xx-us:74S20N
Changed lines of the file:
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@@
 <part name="V4" library="supply2" deviceset="GND" device=""/>
 <part name="V5" library="supply2" deviceset="VCC" device=""/>
-<part name="E4" library="74xx-jameco" deviceset="74*20" device="N" technology="S" value="7440N"/>
-<part name="E3" library="74xx-jameco" deviceset="74*20" device="N" technology="S" value="7440N"/>
+<part name="E4" library="74xx-us" deviceset="74*20" device="N" technology="S" value="7440N"/>
+<part name="E3" library="74xx-us" deviceset="74*20" device="N" technology="S" value="7440N"/>
 <part name="V11" library="supply2" deviceset="VCC" device=""/>
 <part name="V12" library="supply2" deviceset="GND" device=""/>
