File: projects/DEC/Mxxx/M220/M220.sch (EAGLE design)
At the start: 37 parts, among them T1 2N3009B

Commit message: Replace all instances of the 7482 (M220, M221, M222, M628) with one from dec-con, as the standard libraries have all messed up the location of the GND pin.
Parts:
- E13: device 74xx-eu:7482N -> dec-con:7482N
Changed lines of the file:
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@@
 <part name="R2" library="rcl" deviceset="R-US_" device="0207/10" value="180"/>
 <part name="V3" library="supply2" deviceset="VCC" device=""/>
-<part name="E13" library="74xx-eu" deviceset="74*82" device="N"/>
+<part name="E13" library="dec-con" deviceset="74*82" device="N"/>
 <part name="V4" library="supply2" deviceset="GND" device=""/>
 <part name="V5" library="supply2" deviceset="VCC" device=""/>
@@
 </sheet>
 </sheets>
+<errors>
+</errors>
 </schematic>
 </drawing>

Commit message: Where possible, map 74xx-jameco to 74xx-us. Moved the 7438 to dec-con.lbr. Also changed the spelling of CRYTAL to CRYSTAL.
Parts:
- E11, E7: device 74xx-jameco:74S20N -> 74xx-us:74S20N
- E3, E5, E6: device 74xx-jameco:7460N -> 74xx-us:7460N
Changed lines of the file:
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@@
 <part name="V5" library="supply2" deviceset="VCC" device=""/>
 <part name="E1" library="74xxN" deviceset="74*53" device="N"/>
-<part name="E3" library="74xx-jameco" deviceset="74*60" device="N"/>
-<part name="E6" library="74xx-jameco" deviceset="74*60" device="N"/>
+<part name="E3" library="74xx-us" deviceset="74*60" device="N"/>
+<part name="E6" library="74xx-us" deviceset="74*60" device="N"/>
 <part name="E2" library="74xxN" deviceset="74*53" device="N"/>
-<part name="E5" library="74xx-jameco" deviceset="74*60" device="N"/>
+<part name="E5" library="74xx-us" deviceset="74*60" device="N"/>
 <part name="R3" library="rcl" deviceset="R-US_" device="0207/10" value="3K"/>
 <part name="V6" library="supply2" deviceset="VCC" device=""/>
@@
 <part name="V9" library="supply2" deviceset="VCC" device=""/>
 <part name="V10" library="supply2" deviceset="VCC" device=""/>
-<part name="E11" library="74xx-jameco" deviceset="74*20" device="N" technology="S" value="7440N"/>
-<part name="E7" library="74xx-jameco" deviceset="74*20" device="N" technology="S" value="7440N"/>
+<part name="E11" library="74xx-us" deviceset="74*20" device="N" technology="S" value="7440N"/>
+<part name="E7" library="74xx-us" deviceset="74*20" device="N" technology="S" value="7440N"/>
 <part name="V11" library="supply2" deviceset="VCC" device=""/>
 <part name="V12" library="supply2" deviceset="GND" device=""/>

Commit message: Move the various flavors of the 7453 to dec-con.lbr.
Parts:
- E1, E12, E14, E15, E16, E17, E18, E2: device 74xxN:7453N -> dec-con:7453N
Changed lines of the file:
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@@
 <part name="U$1" library="dec-con" deviceset="DOUBLE" device=""/>
 <part name="U$2" library="dec-con" deviceset="OUTLINE-*" device="DOUBLE"/>
-<part name="E12" library="74xxN" deviceset="74*53" device="N"/>
-<part name="E15" library="74xxN" deviceset="74*53" device="N"/>
+<part name="E12" library="dec-con" deviceset="74*53" device="N"/>
+<part name="E15" library="dec-con" deviceset="74*53" device="N"/>
 <part name="V1" library="supply2" deviceset="GND" device=""/>
 <part name="V2" library="supply2" deviceset="VCC" device=""/>
-<part name="E16" library="74xxN" deviceset="74*53" device="N"/>
-<part name="E14" library="74xxN" deviceset="74*53" device="N"/>
-<part name="E18" library="74xxN" deviceset="74*53" device="N"/>
-<part name="E17" library="74xxN" deviceset="74*53" device="N"/>
+<part name="E16" library="dec-con" deviceset="74*53" device="N"/>
+<part name="E14" library="dec-con" deviceset="74*53" device="N"/>
+<part name="E18" library="dec-con" deviceset="74*53" device="N"/>
+<part name="E17" library="dec-con" deviceset="74*53" device="N"/>
 <part name="R1" library="rcl" deviceset="R-US_" device="0207/10" value="180"/>
 <part name="R2" library="rcl" deviceset="R-US_" device="0207/10" value="180"/>
@@
 <part name="V4" library="supply2" deviceset="GND" device=""/>
 <part name="V5" library="supply2" deviceset="VCC" device=""/>
-<part name="E1" library="74xxN" deviceset="74*53" device="N"/>
+<part name="E1" library="dec-con" deviceset="74*53" device="N"/>
 <part name="E3" library="74xx-us" deviceset="74*60" device="N"/>
 <part name="E6" library="74xx-us" deviceset="74*60" device="N"/>
-<part name="E2" library="74xxN" deviceset="74*53" device="N"/>
+<part name="E2" library="dec-con" deviceset="74*53" device="N"/>
 <part name="E5" library="74xx-us" deviceset="74*60" device="N"/>
 <part name="R3" library="rcl" deviceset="R-US_" device="0207/10" value="3K"/>
