File: projects/DEC/Mxxx/M7821/M7821.sch (EAGLE design)
At the start: 58 parts, among them J2 J10MM, J3 J10MM, J4 J10MM, J5 J10MM, J6 J10MM, J7 J10MM, J8 J10MM, J9 J10MM

Commit message: Where possible, map 74xx-jameco to 74xx-us. Moved the 7438 to dec-con.lbr. Also changed the spelling of CRYTAL to CRYSTAL.
Parts:
- E10: device 74xx-jameco:74S08N -> 74xx-us:74S08N
- E12, E18, E5: device 74xx-jameco:74S74N -> 74xx-us:74S74N
- E14, E6: device 74xx-jameco:7402N -> 74xx-us:7402N
- E15, E16, E2, E8, E9: device 74xx-jameco:7438N -> dec-con:7438N
- E17, E4, E7: device 74xx-jameco:7400N -> 74xx-us:7400N
- E3: device 74xx-jameco:74S04N -> 74xx-us:74S04N
Changed lines of the file:
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@@
 <part name="U$1" library="dec-con" deviceset="OUTLINE-*" device="SINGLE-LONG"/>
 <part name="U$2" library="dec-con" deviceset="SINGLE" device=""/>
-<part name="E7" library="74xx-jameco" deviceset="74*00" device="N"/>
+<part name="E7" library="74xx-us" deviceset="74*00" device="N"/>
 <part name="C14" library="rcl" deviceset="C-US" device="050-025X075" value=".01"/>
 <part name="C15" library="rcl" deviceset="C-US" device="050-025X075" value=".01"/>
@@
 <part name="C17" library="rcl" deviceset="C-US" device="050-025X075" value=".01"/>
 <part name="V9" library="supply2" deviceset="GND" device=""/>
-<part name="E9" library="74xx-jameco" deviceset="74*38" device="N"/>
-<part name="E8" library="74xx-jameco" deviceset="74*38" device="N"/>
+<part name="E9" library="dec-con" deviceset="74*38" device="N"/>
+<part name="E8" library="dec-con" deviceset="74*38" device="N"/>
 <part name="J2" library="jumper" deviceset="J" device="10MM"/>
 <part name="J3" library="jumper" deviceset="J" device="10MM"/>
@@
 <part name="J8" library="jumper" deviceset="J" device="10MM"/>
 <part name="J9" library="jumper" deviceset="J" device="10MM"/>
-<part name="E6" library="74xx-jameco" deviceset="74*02" device="N"/>
+<part name="E6" library="74xx-us" deviceset="74*02" device="N"/>
 <part name="R1" library="rcl" deviceset="R-US_" device="0207/10" value="390"/>
 <part name="V10" library="supply2" deviceset="GND" device=""/>
@@
 <part name="R4" library="rcl" deviceset="R-US_" device="0207/10" value="1K"/>
 <part name="V14" library="supply2" deviceset="VCC" device=""/>
-<part name="E18" library="74xx-jameco" deviceset="74*74" device="N" technology="S"/>
-<part name="E12" library="74xx-jameco" deviceset="74*74" device="N" technology="S"/>
-<part name="E5" library="74xx-jameco" deviceset="74*74" device="N" technology="S"/>
-<part name="E10" library="74xx-jameco" deviceset="74*08" device="N" technology="S"/>
-<part name="E3" library="74xx-jameco" deviceset="74*04" device="N" technology="S"/>
+<part name="E18" library="74xx-us" deviceset="74*74" device="N" technology="S"/>
+<part name="E12" library="74xx-us" deviceset="74*74" device="N" technology="S"/>
+<part name="E5" library="74xx-us" deviceset="74*74" device="N" technology="S"/>
+<part name="E10" library="74xx-us" deviceset="74*08" device="N" technology="S"/>
+<part name="E3" library="74xx-us" deviceset="74*04" device="N" technology="S"/>
 <part name="R6" library="rcl" deviceset="R-US_" device="0207/10" value="1K"/>
 <part name="R8" library="rcl" deviceset="R-US_" device="0207/10" value="47"/>
@@
 <part name="E13" library="74xx-us" deviceset="74*02" device="N"/>
 <part name="V8" library="supply2" deviceset="GND" device=""/>
-<part name="E2" library="74xx-jameco" deviceset="74*38" device="N"/>
+<part name="E2" library="dec-con" deviceset="74*38" device="N"/>
 <part name="V2" library="supply2" deviceset="GND" device=""/>
 <part name="V7" library="supply2" deviceset="GND" device=""/>
 <part name="E11" library="dec-con" deviceset="DS8640" device="N"/>
 <part name="FRAME1" library="frames" deviceset="DINA3_L" device=""/>
-<part name="E16" library="74xx-jameco" deviceset="74*38" device="N"/>
+<part name="E16" library="dec-con" deviceset="74*38" device="N"/>
 <part name="V1" library="supply2" deviceset="VCC" device=""/>
-<part name="E15" library="74xx-jameco" deviceset="74*38" device="N"/>
-<part name="E4" library="74xx-jameco" deviceset="74*00" device="N"/>
+<part name="E15" library="dec-con" deviceset="74*38" device="N"/>
+<part name="E4" library="74xx-us" deviceset="74*00" device="N"/>
 <part name="V17" library="supply2" deviceset="VCC" device=""/>
 <part name="V18" library="supply2" deviceset="VCC" device=""/>
-<part name="E17" library="74xx-jameco" deviceset="74*00" device="N"/>
-<part name="E14" library="74xx-jameco" deviceset="74*02" device="N"/>
+<part name="E17" library="74xx-us" deviceset="74*00" device="N"/>
+<part name="E14" library="74xx-us" deviceset="74*02" device="N"/>
 <part name="R5" library="rcl" deviceset="R-US_" device="0207/10" value="180"/>
 <part name="V3" library="supply2" deviceset="VCC" device=""/>
