File: projects/DEC/Rxxx/R210/R210A.brd (EAGLE design)
At the start: 125.7 x 132.1 mm, 228 parts, among them Q1 2N3639, Q10 2N3639, Q11 2N3639, Q12 2N3639, Q2 2N3639, Q3 2N3009, Q4 2N3639, Q5 2N3639, Q6 2N3639, Q7 2N3639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

Commit message: Walk the project tree, making things pass current design rules.
Parts:
- D1, D10, D104, D105, D106, D107, D108, D109, D11, D110, D111, D112, D113, D114, D115, D116, D117, D118, D119, D12, D120, D121, D122, D123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: value 1N4148DO35-10 -> (none)
