File: projects/DEC/VC8x/vc8.sch (EAGLE design)
At the start: 24 parts

Commit message: Remove vestigial use of library dec-r.  Henceforth, dec-m is the library for dec modules.
Parts:
- A04: device dec-r:M101 -> dec-m:M101
- A05: device dec-r:M111 -> dec-m:M111
- A06: device dec-r:M206X -> dec-m:M206X
- A07, A08, A09, A10, B07, B09: device dec-r:M916 -> dec-m:M916
- A11: device dec-r:M921 -> dec-m:M921
- A12: device dec-r:M113 -> dec-m:M113
- B04, B05, B10: device dec-r:M103 -> dec-m:M103
- B06, B08: device dec-r:EMPTY -> dec-m:EMPTY
- B11, B12: device dec-r:M306 -> dec-m:M306
Changed lines of the file:
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@@
 <part name="B02" library="dec-m" deviceset="M903" device=""/>
 <part name="B03" library="dec-m" deviceset="M903" device=""/>
-<part name="B04" library="dec-r" deviceset="M103" device=""/>
-<part name="B05" library="dec-r" deviceset="M103" device=""/>
-<part name="B10" library="dec-r" deviceset="M103" device=""/>
-<part name="B06" library="dec-r" deviceset="EMPTY" device=""/>
-<part name="A07" library="dec-r" deviceset="M916" device="" value="A618A"/>
-<part name="B07" library="dec-r" deviceset="M916" device="" value="A618B"/>
-<part name="A09" library="dec-r" deviceset="M916" device="" value="A618A"/>
-<part name="B09" library="dec-r" deviceset="M916" device="" value="A618B"/>
-<part name="B08" library="dec-r" deviceset="EMPTY" device=""/>
-<part name="A04" library="dec-r" deviceset="M101" device=""/>
-<part name="A05" library="dec-r" deviceset="M111" device=""/>
-<part name="A06" library="dec-r" deviceset="M206X" device="" value="M206"/>
-<part name="A08" library="dec-r" deviceset="M916" device="" value="A702"/>
-<part name="A10" library="dec-r" deviceset="M916" device="" value="A702"/>
-<part name="A11" library="dec-r" deviceset="M921" device=""/>
-<part name="A12" library="dec-r" deviceset="M113" device=""/>
-<part name="B11" library="dec-r" deviceset="M306" device=""/>
-<part name="B12" library="dec-r" deviceset="M306" device=""/>
+<part name="B04" library="dec-m" deviceset="M103" device=""/>
+<part name="B05" library="dec-m" deviceset="M103" device=""/>
+<part name="B10" library="dec-m" deviceset="M103" device=""/>
+<part name="B06" library="dec-m" deviceset="EMPTY" device=""/>
+<part name="A07" library="dec-m" deviceset="M916" device="" value="A618A"/>
+<part name="B07" library="dec-m" deviceset="M916" device="" value="A618B"/>
+<part name="A09" library="dec-m" deviceset="M916" device="" value="A618A"/>
+<part name="B09" library="dec-m" deviceset="M916" device="" value="A618B"/>
+<part name="B08" library="dec-m" deviceset="EMPTY" device=""/>
+<part name="A04" library="dec-m" deviceset="M101" device=""/>
+<part name="A05" library="dec-m" deviceset="M111" device=""/>
+<part name="A06" library="dec-m" deviceset="M206X" device="" value="M206"/>
+<part name="A08" library="dec-m" deviceset="M916" device="" value="A702"/>
+<part name="A10" library="dec-m" deviceset="M916" device="" value="A702"/>
+<part name="A11" library="dec-m" deviceset="M921" device=""/>
+<part name="A12" library="dec-m" deviceset="M113" device=""/>
+<part name="B11" library="dec-m" deviceset="M306" device=""/>
+<part name="B12" library="dec-m" deviceset="M306" device=""/>
 <part name="V1" library="supply2" deviceset="-15V" device=""/>
 <part name="V2" library="supply2" deviceset="GND" device=""/>
@@
 <segment>
 <wire x1="7.62" y1="241.3" x2="20.32" y2="241.3" width="0.1524" layer="91"/>
-<label x="7.62" y="238.76" size="1.778" layer="95"/>
 <label x="7.62" y="241.3" size="1.778" layer="95"/>
 <pinref part="A07" gate="D2" pin="P$2"/>
@@
 <wire x1="7.62" y1="238.76" x2="20.32" y2="238.76" width="0.1524" layer="91"/>
 <pinref part="B07" gate="N2" pin="P$2"/>
+<label x="7.62" y="238.76" size="1.778" layer="95"/>
 </segment>
 </net>
@@
 </sheet>
 </sheets>
+<errors>
+</errors>
 </schematic>
 </drawing>
