File: projects/DEC/Wxxx/W002/W002B.brd (EAGLE design)
At the start: 125.7 x 62.2 mm, 45 parts

Commit message: Walk the project tree, making things pass current design rules.
Connections:
- removed net +10V: U$2.A2
Changed lines of the file:
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@@
 <param name="mdViaViaSameLayer" value="8mil"/>
 <param name="mnLayersViaInSmd" value="2"/>
-<param name="mdCopperDimension" value="25mil"/>
+<param name="mdCopperDimension" value="13mil"/>
 <param name="mdDrill" value="10mil"/>
 <param name="mdSmdStop" value="0mil"/>
@@
 <wire x1="45.72" y1="33.02" x2="48.26" y2="35.56" width="0.8128" layer="16"/>
 </signal>
-<signal name="+10V" class="1">
-<contactref element="U$2" pad="A2"/>
-</signal>
 <signal name="N$1">
