File: projects/ConsoleEmu/core+io4.brd (EAGLE design)
At the start: 215.9 x 107.6 mm, 103 parts, among them IC1 74LS374N, IC10 74154N, IC11 74LS373N, IC12 74LS373N, IC13 74LS373N, IC14 74LS373N, IC15 74LS373N, IC16 74LS373N, IC18 74LS00N, IC19 74LS138N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

Commit message: Walk the project tree, making things pass current design rules.
Connections:
- new net N$139: IC7.2, OUT7-8.2
- net N$26: no longer IC7.2, OUT7-8.2
Routing:
- net N$26: track 93.3 -> 90.1 mm
Changed lines of the file:
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@@
 <wire x1="215.25" y1="107.15" x2="-0.63" y2="107.15" width="0" layer="20"/>
 <wire x1="-0.63" y1="107.15" x2="-0.63" y2="-0.47" width="0" layer="20"/>
+<wire x1="6.35" y1="83.82" x2="8.89" y2="81.28" width="0.4064" layer="21"/>
+<wire x1="8.89" y1="83.82" x2="6.35" y2="81.28" width="0.4064" layer="21"/>
+<wire x1="16.51" y1="81.28" x2="19.05" y2="78.74" width="0.4064" layer="21"/>
+<wire x1="19.05" y1="81.28" x2="16.51" y2="78.74" width="0.4064" layer="21"/>
 </plain>
 <attributes>
@@
 <contactref element="IC5" pad="2"/>
 <contactref element="OUT5-6" pad="2"/>
-<contactref element="IC7" pad="2"/>
-<contactref element="OUT7-8" pad="2"/>
-<wire x1="17.78" y1="57.15" x2="17.78" y2="60.96" width="0.254" layer="1"/>
+<wire x1="17.78" y1="55.88" x2="17.78" y2="60.96" width="0.254" layer="1"/>
 <wire x1="17.78" y1="60.96" x2="16.51" y2="62.23" width="0.254" layer="1"/>
-<wire x1="16.51" y1="62.23" x2="16.51" y2="78.74" width="0.254" layer="1"/>
-<wire x1="16.51" y1="78.74" x2="17.78" y2="80.01" width="0.254" layer="1"/>
-<wire x1="17.78" y1="55.88" x2="17.78" y2="57.15" width="0.254" layer="1"/>
-<wire x1="17.78" y1="80.01" x2="17.78" y2="81.28" width="0.254" layer="1"/>
+<wire x1="16.51" y1="62.23" x2="16.51" y2="78.105" width="0.254" layer="1"/>
+<wire x1="16.51" y1="78.105" x2="17.78" y2="79.375" width="0.254" layer="1"/>
 <wire x1="7.62" y1="59.055" x2="6.35" y2="60.325" width="0.254" layer="1"/>
 <wire x1="6.35" y1="60.325" x2="6.35" y2="77.47" width="0.254" layer="1"/>
 <wire x1="6.35" y1="77.47" x2="7.62" y2="78.74" width="0.254" layer="1"/>
-<wire x1="7.62" y1="78.74" x2="7.62" y2="83.185" width="0.254" layer="1"/>
+<wire x1="7.62" y1="78.74" x2="7.62" y2="82.55" width="0.254" layer="1"/>
 <wire x1="7.62" y1="58.42" x2="7.62" y2="59.055" width="0.254" layer="1"/>
-<wire x1="7.62" y1="83.185" x2="7.62" y2="83.82" width="0.254" layer="1"/>
-<wire x1="15.875" y1="53.975" x2="17.145" y2="55.245" width="0.254" layer="16"/>
+<wire x1="15.875" y1="53.975" x2="17.78" y2="55.88" width="0.254" layer="16"/>
 <wire x1="8.89" y1="53.975" x2="15.875" y2="53.975" width="0.254" layer="16"/>
 <wire x1="5.08" y1="57.785" x2="8.89" y2="53.975" width="0.254" layer="16"/>
@@
 <wire x1="6.35" y1="61.595" x2="6.35" y2="59.055" width="0.254" layer="16"/>
 <wire x1="6.35" y1="59.055" x2="7.62" y2="59.055" width="0.254" layer="16"/>
-<wire x1="17.145" y1="55.245" x2="17.78" y2="55.88" width="0.254" layer="16"/>
 <wire x1="7.62" y1="59.055" x2="7.62" y2="58.42" width="0.254" layer="16"/>
 </signal>
@@
 <wire x1="140.335" y1="24.765" x2="140.97" y2="25.4" width="0.254" layer="1"/>
 </signal>
+<signal name="N$139">
+<contactref element="IC7" pad="2"/>
+<contactref element="OUT7-8" pad="2"/>
+<wire x1="7.62" y1="83.82" x2="17.78" y2="81.28" width="0" layer="19" extent="1-1"/>
+</signal>
 </signals>
