File: projects/ConsoleEmu/core5.sch (EAGLE design)
At the start: 59 parts, among them IC17 6802, IC18 74LS132N, IC19 74LS138N, IC20 MAX232, IC21 6850, IC22 6264A, IC23 27C128P, IC24 6821, IC25 74LS245N, IC26 74LS245N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

Commit message: Where possible, map 74xx-jameco to 74xx-us. Moved the 7438 to dec-con.lbr. Also changed the spelling of CRYTAL to CRYSTAL.
Parts:
- Q1: device crystal:CRYTALHC18U-V -> crystal:CRYSTALHC18U-V
Changed lines of the file:
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@@
 <parts>
 <part name="IC17" library="micro-motorola" deviceset="6802" device="" value="6802"/>
-<part name="Q1" library="crystal" deviceset="CRYTAL" device="HC18U-V" value="4Mhz"/>
+<part name="Q1" library="crystal" deviceset="CRYSTAL" device="HC18U-V" value="4Mhz"/>
 <part name="C1" library="rcl" deviceset="C-US" device="050-025X075" value="27pf"/>
 <part name="C2" library="rcl" deviceset="C-US" device="050-025X075" value="27pf"/>
