File: projects/FlipChipTester/tester-rp.sch (EAGLE design)
At the start: 54 parts, among them IC1 74LS125N, IC2 74LS125N, IC3 74LS125N, IC4 74LS125N, IC5 74LS125N, IC6 74LS125N, IC7 74LS125N, IC8 74LS125N, IC9 74LS00N

Commit message: Where possible, map 74xx-jameco to 74xx-us. Moved the 7438 to dec-con.lbr. Also changed the spelling of CRYTAL to CRYSTAL.
Parts:
- IC1, IC2, IC3, IC4, IC5, IC6, IC7, IC8: device 74xx-jameco:74LS125N -> 74xx-us:74LS125N
- IC9: device 74xx-jameco:74LS00N -> 74xx-us:74LS00N
Changed lines of the file:
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@@
 <part name="V19" library="supply2" deviceset="GND" device=""/>
 <part name="POWER" library="jumper" deviceset="JP1Q" device="" value="POWER"/>
-<part name="IC1" library="74xx-jameco" deviceset="74*125" device="N" technology="LS"/>
-<part name="IC2" library="74xx-jameco" deviceset="74*125" device="N" technology="LS"/>
+<part name="IC1" library="74xx-us" deviceset="74*125" device="N" technology="LS"/>
+<part name="IC2" library="74xx-us" deviceset="74*125" device="N" technology="LS"/>
 <part name="OUT5-6" library="con-lstb" deviceset="MA08-2" device=""/>
-<part name="IC5" library="74xx-jameco" deviceset="74*125" device="N" technology="LS"/>
-<part name="IC6" library="74xx-jameco" deviceset="74*125" device="N" technology="LS"/>
+<part name="IC5" library="74xx-us" deviceset="74*125" device="N" technology="LS"/>
+<part name="IC6" library="74xx-us" deviceset="74*125" device="N" technology="LS"/>
 <part name="OUT3-4" library="con-lstb" deviceset="MA08-2" device=""/>
-<part name="IC3" library="74xx-jameco" deviceset="74*125" device="N" technology="LS"/>
-<part name="IC4" library="74xx-jameco" deviceset="74*125" device="N" technology="LS"/>
+<part name="IC3" library="74xx-us" deviceset="74*125" device="N" technology="LS"/>
+<part name="IC4" library="74xx-us" deviceset="74*125" device="N" technology="LS"/>
 <part name="OUT7-8" library="con-lstb" deviceset="MA08-2" device=""/>
-<part name="IC7" library="74xx-jameco" deviceset="74*125" device="N" technology="LS"/>
-<part name="IC8" library="74xx-jameco" deviceset="74*125" device="N" technology="LS"/>
+<part name="IC7" library="74xx-us" deviceset="74*125" device="N" technology="LS"/>
+<part name="IC8" library="74xx-us" deviceset="74*125" device="N" technology="LS"/>
 <part name="CORE-IO" library="con-lstb" deviceset="MA10-2" device=""/>
-<part name="IC9" library="74xx-jameco" deviceset="74*00" device="N" technology="LS"/>
+<part name="IC9" library="74xx-us" deviceset="74*00" device="N" technology="LS"/>
 <part name="C1" library="rcl" deviceset="C-US" device="050-025X075" value="0.1uf"/>
 <part name="V1" library="supply2" deviceset="GND" device=""/>

Commit message: Walk the project tree, making things pass current design rules.
Changed lines of the file:
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@@
 <pinref part="IC9" gate="C" pin="O"/>
 <pinref part="OC" gate="G$1" pin="1"/>
+<label x="269.24" y="66.04" size="1.778" layer="95" rot="R90"/>
 </segment>
 <segment>
@@
 <pinref part="IC9" gate="D" pin="O"/>
 <pinref part="!MR" gate="G$1" pin="1"/>
+<label x="269.24" y="81.28" size="1.778" layer="95" rot="R90"/>
 </segment>
 </net>
@@
 </sheet>
 </sheets>
+<errors>
+</errors>
 </schematic>
 </drawing>
