File: projects/For Zane/1541-3m.sch (EAGLE design)
At the start: 79 parts, among them IC2 MAX702CPA, IC3 PIC18F252I/SP, IC4 MAX232, J1 SDCARDMOUSER, J2 Dev8/Dev9, J3 Boot/Norm, P1 1K, X1 20Mhz

Commit message: Where possible, map 74xx-jameco to 74xx-us. Moved the 7438 to dec-con.lbr. Also changed the spelling of CRYTAL to CRYSTAL.
Parts:
- X1: device crystal:CRYTALHC49U70 -> crystal:CRYSTALHC49U70
Changed lines of the file:
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@@
 <part name="AC2" library="wirepad" deviceset="2,15/1,0" device=""/>
 <part name="AC1" library="wirepad" deviceset="2,15/1,0" device=""/>
-<part name="X1" library="crystal" deviceset="CRYTAL" device="HC49U70" value="20Mhz"/>
+<part name="X1" library="crystal" deviceset="CRYSTAL" device="HC49U70" value="20Mhz"/>
 <part name="R24" library="rcl" deviceset="R-US_" device="0207/2V" value="10"/>
 <part name="C14" library="rcl" deviceset="C-US" device="025-024X044" value="15pf"/>

Commit message: Walk the project tree, making things pass current design rules.
Parts:
- D3-7: value (none) -> R1BA
- IC1, IC5: value (none) -> LM317TS
Changed lines of the file:
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@@
 <part name="V19" library="supply2" deviceset="VCC" device=""/>
 <part name="V20" library="supply2" deviceset="GND" device=""/>
-<part name="D3-7" library="rectifier" deviceset="RB1A" device=""/>
+<part name="D3-7" library="rectifier" deviceset="RB1A" device="" value="R1BA"/>
 <part name="AC2" library="wirepad" deviceset="2,15/1,0" device=""/>
 <part name="AC1" library="wirepad" deviceset="2,15/1,0" device=""/>
@@
 <part name="R11" library="rcl" deviceset="R-US_" device="0207/2V" value="200"/>
 <part name="R12" library="rcl" deviceset="R-US_" device="0207/2V" value="330"/>
-<part name="IC1" library="v-reg" deviceset="LM317TS" device=""/>
-<part name="IC5" library="v-reg" deviceset="LM317TS" device=""/>
+<part name="IC1" library="v-reg" deviceset="LM317TS" device="" value="LM317TS"/>
+<part name="IC5" library="v-reg" deviceset="LM317TS" device="" value="LM317TS"/>
 <part name="C6" library="rcl" deviceset="C-US" device="025-024X044" value=".01uf"/>
 <part name="V39" library="supply2" deviceset="GND" device=""/>
@@
 </sheet>
 </sheets>
+<errors>
+</errors>
 </schematic>
 </drawing>
