File: projects/mmu6100/vrs6907.sch (EAGLE design)
At the start: 54 parts, among them IC1 74LS74N, IC2 74HCT374N, IC3 7407N, IC4 74LS32N, IC6 74LS74N, IC7 74LS10N

Commit message: Where possible, map 74xx-jameco to 74xx-us. Moved the 7438 to dec-con.lbr. Also changed the spelling of CRYTAL to CRYSTAL.
Parts:
- 3B: device 74xx-jameco:7414N -> 74xx-us:7414N
- 3D, IC1, IC6: device 74xx-jameco:74LS74N -> 74xx-us:74LS74N
- 3E, IC7: device 74xx-jameco:74LS10N -> 74xx-us:74LS10N
- 3F: device 74xx-jameco:74LS00N -> 74xx-us:74LS00N
- 4A: value 74HCT138N -> 74LS138N; device 74xx-jameco:74HCT138N -> 74xx-us:74LS138N
- 4B, 6F: device 74xx-jameco:74LS174N -> 74xx-us:74LS174N
- 4D, 5B, 5C: device 74xx-jameco:74LS175N -> 74xx-us:74LS175N
- 4E: device 74xx-jameco:74LS02N -> 74xx-us:74LS02N
- 4F: device 74xx-jameco:74LS04N -> 74xx-us:74LS04N
- 5D: device 74xx-jameco:74LS257N -> 74xx-us:74LS257N
- 5E, IC3: device 74xx-jameco:7407N -> 74xx-us:7407N
- 5F, IC4: device 74xx-jameco:74LS32N -> 74xx-us:74LS32N
- 6B, 6C, 6D, 6E: device 74xx-jameco:74LS365N -> 74xx-us:74LS365N
- IC2: value 74HCT374N -> 74LS374N; device 74xx-jameco:74HCT374N -> 74xx-us:74LS374N
Changed lines of the file:
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@@
 <parts>
 <part name="FRAME1" library="frames" deviceset="DINA3_L" device=""/>
-<part name="3B" library="74xx-jameco" deviceset="74*14" device="N"/>
-<part name="5E" library="74xx-jameco" deviceset="74*07" device="N"/>
-<part name="4F" library="74xx-jameco" deviceset="74*04" device="N" technology="LS"/>
-<part name="4E" library="74xx-jameco" deviceset="74*02" device="N" technology="LS"/>
-<part name="3F" library="74xx-jameco" deviceset="74*00" device="N" technology="LS"/>
-<part name="3D" library="74xx-jameco" deviceset="74*74" device="N" technology="LS"/>
+<part name="3B" library="74xx-us" deviceset="74*14" device="N"/>
+<part name="5E" library="74xx-us" deviceset="74*07" device="N"/>
+<part name="4F" library="74xx-us" deviceset="74*04" device="N" technology="LS"/>
+<part name="4E" library="74xx-us" deviceset="74*02" device="N" technology="LS"/>
+<part name="3F" library="74xx-us" deviceset="74*00" device="N" technology="LS"/>
+<part name="3D" library="74xx-us" deviceset="74*74" device="N" technology="LS"/>
 <part name="V1" library="supply2" deviceset="VCC" device=""/>
-<part name="6E" library="74xx-jameco" deviceset="74*365" device="N" technology="LS"/>
+<part name="6E" library="74xx-us" deviceset="74*365" device="N" technology="LS"/>
 <part name="V2" library="supply2" deviceset="GND" device=""/>
-<part name="5F" library="74xx-jameco" deviceset="74*32" device="N" technology="LS"/>
-<part name="6F" library="74xx-jameco" deviceset="74*174" device="N" technology="LS"/>
+<part name="5F" library="74xx-us" deviceset="74*32" device="N" technology="LS"/>
+<part name="6F" library="74xx-us" deviceset="74*174" device="N" technology="LS"/>
 <part name="V4" library="supply2" deviceset="VCC" device=""/>
-<part name="4B" library="74xx-jameco" deviceset="74*174" device="N" technology="LS"/>
+<part name="4B" library="74xx-us" deviceset="74*174" device="N" technology="LS"/>
 <part name="C1" library="rcl" deviceset="CPOL-US" device="E22-6AXIAL" value="27uf"/>
 <part name="C2" library="rcl" deviceset="CPOL-US" device="E22-6AXIAL" value="27uf"/>
 <part name="V3" library="supply2" deviceset="GND" device=""/>
 <part name="V5" library="supply2" deviceset="VCC" device=""/>
-<part name="6C" library="74xx-jameco" deviceset="74*365" device="N" technology="LS"/>
-<part name="5C" library="74xx-jameco" deviceset="74*175" device="N" technology="LS"/>
-<part name="5B" library="74xx-jameco" deviceset="74*175" device="N" technology="LS"/>
-<part name="6B" library="74xx-jameco" deviceset="74*365" device="N" technology="LS"/>
-<part name="4D" library="74xx-jameco" deviceset="74*175" device="N" technology="LS"/>
-<part name="6D" library="74xx-jameco" deviceset="74*365" device="N" technology="LS"/>
+<part name="6C" library="74xx-us" deviceset="74*365" device="N" technology="LS"/>
+<part name="5C" library="74xx-us" deviceset="74*175" device="N" technology="LS"/>
+<part name="5B" library="74xx-us" deviceset="74*175" device="N" technology="LS"/>
+<part name="6B" library="74xx-us" deviceset="74*365" device="N" technology="LS"/>
+<part name="4D" library="74xx-us" deviceset="74*175" device="N" technology="LS"/>
+<part name="6D" library="74xx-us" deviceset="74*365" device="N" technology="LS"/>
 <part name="V7" library="supply2" deviceset="VCC" device=""/>
-<part name="5D" library="74xx-jameco" deviceset="74*257" device="N" technology="LS"/>
-<part name="3E" library="74xx-jameco" deviceset="74*10" device="N" technology="LS"/>
+<part name="5D" library="74xx-us" deviceset="74*257" device="N" technology="LS"/>
+<part name="3E" library="74xx-us" deviceset="74*10" device="N" technology="LS"/>
 <part name="V8" library="supply2" deviceset="VCC" device=""/>
 <part name="V10" library="supply2" deviceset="GND" device=""/>
@@
 <part name="R2" library="rcl" deviceset="R-US_" device="0207/10"/>
 <part name="V6" library="supply2" deviceset="VCC" device=""/>
-<part name="4A" library="74xx-jameco" deviceset="74*138" device="N" technology="HCT"/>
+<part name="4A" library="74xx-us" deviceset="74*138" device="N" technology="LS" value="74LS138N"/>
 <part name="V17" library="supply2" deviceset="VCC" device=""/>
-<part name="IC7" library="74xx-jameco" deviceset="74*10" device="N" technology="LS"/>
-<part name="IC6" library="74xx-jameco" deviceset="74*74" device="N" technology="LS"/>
+<part name="IC7" library="74xx-us" deviceset="74*10" device="N" technology="LS"/>
+<part name="IC6" library="74xx-us" deviceset="74*74" device="N" technology="LS"/>
 <part name="V18" library="supply2" deviceset="GND" device=""/>
-<part name="IC3" library="74xx-jameco" deviceset="74*07" device="N"/>
-<part name="IC4" library="74xx-jameco" deviceset="74*32" device="N" technology="LS"/>
-<part name="IC1" library="74xx-jameco" deviceset="74*74" device="N" technology="LS"/>
+<part name="IC3" library="74xx-us" deviceset="74*07" device="N"/>
+<part name="IC4" library="74xx-us" deviceset="74*32" device="N" technology="LS"/>
+<part name="IC1" library="74xx-us" deviceset="74*74" device="N" technology="LS"/>
 <part name="V23" library="supply2" deviceset="VCC" device=""/>
-<part name="IC2" library="74xx-jameco" deviceset="74*374" device="N" technology="HCT"/>
+<part name="IC2" library="74xx-us" deviceset="74*374" device="N" technology="LS" value="74LS374N"/>
 <part name="V9" library="supply2" deviceset="GND" device=""/>
 <part name="SV1" library="con-lstb" deviceset="MA03-1" device=""/>
