File: projects/DEC/DW08A/dw08a2s.brd (EAGLE design)
At the start: 319.1 x 141 mm, 48 parts

Commit message: Clean up DW08 Udrawings which were refusing to update (replaced the obsolete parts manually).
Routing:
- net GND: track 2824.9 -> 2829.0 mm
