File: projects/DEC/Mxxx/M228/M228A.brd (EAGLE design)
At the start: 125.7 x 132.1 mm, 52 parts

Commit message: Move 7450 to dec-con and fix all references to it.
Parts:
- E7: device 74xxN:DIL14 -> dec-con:DIL14
Changed lines of the file:
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@@
 <element name="E21" library="74xx-us" package="DIL14" value="7430N" x="30.48" y="16.51"/>
 <element name="E19" library="74xxN" package="DIL14" value="7453N" x="93.98" y="16.51"/>
-<element name="E7" library="74xxN" package="DIL14" value="7450N" x="93.98" y="82.55"/>
+<element name="E7" library="dec-con" package="DIL14" value="7450N" x="93.98" y="82.55"/>
 <element name="C19" library="rcl" package="C050-025X075" value=".01uf" x="74.93" y="15.24" rot="R270"/>
 <element name="C20" library="rcl" package="C050-025X075" value=".01uf" x="49.53" y="12.7" rot="R270"/>

Commit message: Walk the project tree, making things pass current design rules.
Routing:
- net AU1: track 210.0 -> 210.7 mm
Changed lines of the file:
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@@
 <setting verticaltext="up"/>
 </settings>
-<grid distance="0.05" unitdist="inch" unit="inch" style="dots" multiple="2" display="yes" altdistance="10" altunitdist="mil" altunit="mil"/>
+<grid distance="0.05" unitdist="inch" unit="inch" style="dots" multiple="2" display="yes" altdistance="25" altunitdist="mil" altunit="mil"/>
 <layers>
 <layer number="1" name="Top" color="4" fill="1" visible="yes" active="yes"/>
@@
 <param name="mdViaViaSameLayer" value="8mil"/>
 <param name="mnLayersViaInSmd" value="2"/>
-<param name="mdCopperDimension" value="25mil"/>
+<param name="mdCopperDimension" value="13mil"/>
 <param name="mdDrill" value="10mil"/>
 <param name="mdSmdStop" value="0mil"/>
@@
 <wire x1="99.06" y1="64.77" x2="101.6" y2="62.23" width="0.8128" layer="16"/>
 <wire x1="116.84" y1="52.07" x2="117.7925" y2="51.7525" width="0.8128" layer="16"/>
-<wire x1="111.76" y1="52.07" x2="116.84" y2="52.07" width="0.8128" layer="16"/>
-<wire x1="107.95" y1="57.15" x2="111.76" y2="52.07" width="0.8128" layer="16"/>
+<wire x1="111.125" y1="52.07" x2="116.84" y2="52.07" width="0.8128" layer="16"/>
+<wire x1="107.95" y1="57.15" x2="111.125" y2="52.07" width="0.8128" layer="16"/>
 <wire x1="102.87" y1="62.23" x2="107.95" y2="57.15" width="0.8128" layer="16"/>
 <wire x1="101.6" y1="62.23" x2="102.87" y2="62.23" width="0.8128" layer="16"/>
@@
 <wire x1="80.01" y1="43.18" x2="83.82" y2="41.91" width="0.4064" layer="16"/>
 <wire x1="116.84" y1="41.91" x2="117.7925" y2="42.2275" width="0.4064" layer="16"/>
-<wire x1="111.76" y1="41.91" x2="116.84" y2="41.91" width="0.4064" layer="16"/>
-<wire x1="109.22" y1="39.37" x2="111.76" y2="41.91" width="0.4064" layer="16"/>
+<wire x1="111.125" y1="41.91" x2="116.84" y2="41.91" width="0.4064" layer="16"/>
+<wire x1="109.22" y1="39.37" x2="111.125" y2="41.91" width="0.4064" layer="16"/>
 <wire x1="106.68" y1="39.37" x2="109.22" y2="39.37" width="0.4064" layer="16"/>
 <wire x1="104.14" y1="41.91" x2="106.68" y2="39.37" width="0.4064" layer="16"/>
@@
 <contactref element="U$5" pad="AR2"/>
 <wire x1="116.84" y1="86.36" x2="117.7925" y2="86.6775" width="0.4064" layer="16"/>
-<wire x1="111.76" y1="86.36" x2="116.84" y2="86.36" width="0.4064" layer="16"/>
-<wire x1="109.22" y1="83.82" x2="111.76" y2="86.36" width="0.4064" layer="16"/>
-<wire x1="104.14" y1="83.82" x2="109.22" y2="83.82" width="0.4064" layer="16"/>
+<wire x1="110.49" y1="86.36" x2="116.84" y2="86.36" width="0.4064" layer="16"/>
+<wire x1="107.95" y1="83.82" x2="110.49" y2="86.36" width="0.4064" layer="16"/>
+<wire x1="104.14" y1="83.82" x2="107.95" y2="83.82" width="0.4064" layer="16"/>
 <wire x1="104.14" y1="83.82" x2="91.44" y2="83.82" width="0.4064" layer="16"/>
 <wire x1="91.44" y1="83.82" x2="88.9" y2="86.36" width="0.4064" layer="16"/>
@@
 <wire x1="78.74" y1="59.69" x2="77.47" y2="60.96" width="0.4064" layer="1"/>
 <wire x1="116.84" y1="77.47" x2="117.7925" y2="77.1525" width="0.4064" layer="1"/>
-<wire x1="111.76" y1="77.47" x2="116.84" y2="77.47" width="0.4064" layer="1"/>
-<wire x1="106.68" y1="82.55" x2="111.76" y2="77.47" width="0.4064" layer="1"/>
-<wire x1="106.68" y1="85.09" x2="106.68" y2="82.55" width="0.4064" layer="1"/>
+<wire x1="110.49" y1="77.47" x2="116.84" y2="77.47" width="0.4064" layer="1"/>
+<wire x1="106.68" y1="81.28" x2="110.49" y2="77.47" width="0.4064" layer="1"/>
+<wire x1="106.68" y1="85.09" x2="106.68" y2="81.28" width="0.4064" layer="1"/>
 <wire x1="100.33" y1="91.44" x2="106.68" y2="85.09" width="0.4064" layer="1"/>
 <wire x1="90.17" y1="91.44" x2="100.33" y2="91.44" width="0.4064" layer="1"/>

Commit message: Move the various flavors of the 7453 to dec-con.lbr.
Parts:
- E19: device 74xxN:DIL14 -> dec-con:DIL14
Changed lines of the file:
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@@
 <element name="E2" library="74xx-us" package="DIL14" value="7430N" x="62.23" y="115.57"/>
 <element name="E21" library="74xx-us" package="DIL14" value="7430N" x="30.48" y="16.51"/>
-<element name="E19" library="74xxN" package="DIL14" value="7453N" x="93.98" y="16.51"/>
+<element name="E19" library="dec-con" package="DIL14" value="7453N" x="93.98" y="16.51"/>
 <element name="E7" library="dec-con" package="DIL14" value="7450N" x="93.98" y="82.55"/>
 <element name="C19" library="rcl" package="C050-025X075" value=".01uf" x="74.93" y="15.24" rot="R270"/>
