File: projects/PLD-Omnibus/M8357pld.brd (EAGLE design)
At the start: 265.3 x 214.6 mm, 47 parts

Commit message: Finish fixing "no such part in library" stuff.
Parts:
- E1: value ATF1508PQFP -> ATF150X100PQFP
Changed lines of the file:
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@@
 <element name="C44" library="rcl" package="E22-6" value="6.8uf" x="186.69" y="35.56" rot="R180"/>
 <element name="C45" library="rcl" package="E22-6" value="6.8uf" x="237.49" y="35.56" rot="R180"/>
-<element name="E1" library="atmel-cpld" package="PQFP-100" value="ATF1508PQFP" x="73.66" y="88.9"/>
+<element name="E1" library="atmel-cpld" package="PQFP-100" value="ATF150X100PQFP" x="73.66" y="88.9"/>
 <element name="ISP" library="con-lstb" package="MA05-2" value="" x="92.71" y="114.3" rot="R90">
 <attribute name="OC_NEWARK" value="unknown" x="92.71" y="114.3" size="1.778" layer="27" rot="R90" display="off"/>

Commit message: Check in breakout boards for 100 pin Atmel CPLDs. Update Omnibus CPLD work to reflect library pin changes. Fix Omnibus pin polarity for active low signals in the CPLD designs.
Parts:
- ISP: device con-lstb:MA05-2 -> con-ml:ML10
- moved ISP 75.5 mm to (83.8, 189.2), turned to 0 degrees
Connections:
- net !C0: now also E1.25; no longer E1.23
- net !C1: now also E1.24; no longer E1.22
- net !DATA0: now also E1.46; no longer E1.42
- net !DATA1: now also E1.44; no longer E1.39
- net !DATA10: now also E1.7; no longer E1.2
- net !DATA11: now also E1.4; no longer E1.1
- net !DATA2: now also E1.42; no longer E1.38
- net !DATA3: now also E1.39; no longer E1.37
- net !DATA4: now also E1.33; no longer E1.31
- net !DATA5: now also E1.32; no longer E1.30
- net !DATA6: now also E1.31; no longer E1.29
- net !DATA7: now also E1.29; no longer E1.26
- net !DATA8: now also E1.8; no longer E1.4
- net !DONE_SKIP: now also E1.62; no longer E1.59
- net !INTERNAL_IO: now also E1.21; no longer E1.18
- net !INT_RQST: now also E1.16; no longer E1.14
- net !IO_PAUSE: now also E1.26; no longer E1.24
- net !MD03: now also E1.47; no longer E1.44
- net !MD04: now also E1.38; no longer E1.35
- net !MD05: now also E1.37; no longer E1.34
- net !MD06: now also E1.35; no longer E1.33
- net !MD07: now also E1.34; no longer E1.32
- net !MD08: now also E1.12; no longer E1.10
- net !MD09: now also E1.11; no longer E1.9
- net !MD10: now also E1.10; no longer E1.8
- net !MD11: now also E1.9; no longer E1.7
- net !RX_12_BIT: now also E1.86; no longer E1.83
- net !RX_DATA: now also E1.83; no longer E1.81
- net !RX_DONE: now also E1.81; no longer E1.79
- net !RX_ERROR: now also E1.74; no longer E1.72
- net !RX_INIT: now also E1.78; no longer E1.74
- net !RX_OUT: now also E1.1; no longer E1.99
- net !RX_RUN: now also E1.72; no longer E1.70
- net !RX_SHIFT: now also E1.99; no longer E1.96
- net !RX_TR_REQ: now also E1.79; no longer E1.77
- net !SKIP: now also E1.14; no longer E1.11
- net !TR_SKIP: now also E1.63; no longer E1.60
- net INITIALIZE: now also E1.15; no longer E1.12
- net N$7: now also E1.94; no longer E1.85
- net N$8: now also E1.95; no longer E1.86
- net N$9: now also E1.96; no longer E1.94
- net PARITY: now also E1.60; no longer E1.58
- net TP3: now also E1.23; no longer E1.21
- net TP4: now also E1.22; no longer E1.19
Routing:
- net GND: track 170.3 -> 956.0 mm, vias 9 -> 3
- net VCC: track 134.4 -> 553.4 mm, vias 2 -> 5
- net PARITY: track 222.3 -> 309.2 mm, vias 2 -> 0
- net TDO: track 33.3 -> 118.3 mm, vias 1 -> 3
- net TMS: track 48.3 -> 123.9 mm, vias 2 -> 1
- net TCK: track 26.3 -> 92.7 mm, vias 1 -> 0
- net TDI: track 66.2 -> 126.9 mm, vias 2 -> 3
- net !MD07: track 211.1 -> 178.0 mm
- net !DATA1: track 196.1 -> 172.8 mm
- net !MD05: track 137.1 -> 158.6 mm, vias 2 -> 0
- net N$9: track 66.8 -> 46.4 mm, vias 1 -> 0
- net !RX_DONE: track 95.4 -> 111.3 mm, vias 1 -> 0
- net N$6: track 56.9 -> 41.3 mm, vias 1 -> 2
- net !RX_ERROR: track 116.1 -> 131.1 mm
- net !RX_TR_REQ: track 114.1 -> 103.3 mm, vias 0 -> 1
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