File: projects/X8iPanel/LEDpanelmpsl.brd (EAGLE design)
At the start: 377.8 x 138.1 mm, 297 parts

Commit message: Walk the project tree, making things pass current design rules.
Parts:
- turned T1 to 0 degrees
- turned T10 to 0 degrees
- turned T11 to 0 degrees
- turned T12 to 0 degrees
- turned T13 to 0 degrees
- turned T14 to 0 degrees
- turned T15 to 0 degrees
- turned T16 to 0 degrees
- turned T17 to 0 degrees
- turned T18 to 0 degrees
- turned T19 to 90 degrees
- turned T2 to 0 degrees
- turned T20 to 90 degrees
- turned T21 to 90 degrees
- turned T22 to 90 degrees
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Routing:
- net GND: track 2842.7 -> 2324.2 mm
- net N$71: track 9.53 -> 4.45 mm
- net N$69: track 9.53 -> 4.45 mm
- net N$67: track 9.53 -> 4.45 mm
- net N$66: track 9.53 -> 4.45 mm
- net N$64: track 9.53 -> 4.45 mm
- net N$62: track 9.53 -> 4.45 mm
- net N$60: track 9.53 -> 4.45 mm
- net N$58: track 9.53 -> 4.45 mm
- net N$56: track 9.53 -> 4.45 mm
- net N$72: track 9.52 -> 4.45 mm
- net N$54: track 9.52 -> 4.45 mm
- net N$52: track 9.52 -> 4.45 mm
- net N$50: track 9.52 -> 4.45 mm
- net N$48: track 9.52 -> 4.45 mm
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
Commit message: Update 8/I lights boards to fix bulb placement based on feedback from Oscar.
Parts:
- moved DCA 2.25 mm to (306.4, 65.1)
- moved DEFER 2.25 mm to (335.0, 76.2)
- moved EXECUTE 2.25 mm to (335.0, 87.3)
- moved ISZ 2.25 mm to (306.4, 76.2)
- moved R76 2.25 mm to (329.9, 95.2)
- moved R77 2.25 mm to (329.9, 84.1)
- moved R78 2.25 mm to (329.9, 73.0)
- moved T76 2.25 mm to (342.9, 100.0)
- moved T77 2.25 mm to (342.9, 88.9)
- moved T81 2.25 mm to (342.9, 44.5)
- moved T82 2.25 mm to (314.3, 100.0)
- moved T83 2.25 mm to (314.3, 88.9)
- moved T87 2.25 mm to (314.3, 44.5)
- moved TAD 2.25 mm to (306.4, 87.3)
- moved WORDCOUNT 2.25 mm to (335.0, 65.1)
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Routing:
- net GND: track 2324.2 -> 2302.7 mm
- net N$12: track 20.3 -> 5.79 mm
- net +15V: track 1892.4 -> 1878.3 mm
- net MQ6: track 124.0 -> 131.7 mm
- net N$101: track 13.8 -> 7.01 mm
- net IF1: track 212.1 -> 206.7 mm
- net TAD: track 42.8 -> 37.7 mm
- net MQ11: track 128.2 -> 123.9 mm
- net MQ5: track 124.3 -> 121.1 mm
- net AC5: track 106.4 -> 103.2 mm
- net MB5: track 105.5 -> 102.3 mm
- net AC0: track 93.7 -> 96.2 mm
- net AND: track 28.3 -> 26.0 mm
- net MQ7: track 118.7 -> 121.0 mm
- net MB4: track 65.8 -> 63.6 mm
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Other:
- board size 377.8 x 138.1 mm -> 377.8 x 165.1 mm
