File: projects/X8iPanel/8iPanelDec.sch (EAGLE design)
At the start: 194 parts, among them T1 2N2222, T10 2N2222, T11 2N2222, T12 2N2222, T13 2N2222, T14 2N2222, T15 2N2222, T16 2N2222, T17 2N2222, T18 2N2222, T19 2N2222, T2 2N2222, T20 2N2222, T21 2N2222, T22 2N2222, T23 2N2222, T24 2N2222, T25 2N2222, T26 2N2222, T27 2N2222, T28 2N2222, T29 2N2222, T3 2N2222, T30 2N2222, T31 2N2222, T32 2N2222, T33 2N2222, T34 2N2222, T35 2N2222, T36 2N2222, T37 2N2222, T38 2N2222, T39 2N2222, T4 2N2222, T40 2N2222, T41 2N2222, T42 2N2222, T43 2N2222, T44 2N2222, T45 2N2222, T46 2N2222, T47 2N2222, T48 2N2222, T49 2N2222, T5 2N2222, T50 2N2222, T51 2N2222, T52 2N2222, T53 2N2222, T54 2N2222, T55 2N2222, T56 2N2222, T57 2N2222, T58 2N2222, T59 2N2222, T6 2N2222, T60 2N2222, T61 2N2222, T62 2N2222, T63 2N2222, T64 2N2222, T65 2N2222, T66 2N2222, T67 2N2222, T68 2N2222, T69 2N2222, T7 2N2222, T70 2N2222, T71 2N2222, T72 2N2222, T73 2N2222, T74 2N2222, T75 2N2222, T76 2N2222, T77 2N2222, T78 2N2222, T79 2N2222, T8 2N2222, T80 2N2222, T81 2N2222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

Commit message: Fix wiring errors in 8iPanelDec drawings.
Parts:
- removed +15V1, +15V2, GND1, GND2, X1, X2, X3, X4: 494864, con-ptr500:AK500/2
- added +15V, GND, NC1, NC2: LUG, dec-con:LUG
Connections:
- net +15V: now also +15V.1; no longer +15V1-1.KL, +15V1-2.KL, +15V2-1.KL, +15V2-2.KL, X1-1.KL, X1-2.KL, X2-1.KL, X2-2.KL
- net AC0: now also E40TOP4.1; no longer D40TOP4.1
- net AC1: now also E40BOT2.1; no longer D40BOT2.1
- net AC10: now also F40TOP17.1; no longer E40TOP17.1
- net AC11: now also F40BOT16.1; no longer E40BOT16.1
- net AC2: now also E40TOP12.1; no longer D40TOP12.1
- net AC3: now also E40BOT9.1; no longer D40BOT9.1
- net AC4: now also E40TOP17.1; no longer D40TOP17.1
- net AC5: now also E40BOT16.1; no longer D40BOT16.1
- net AC6: now also F40TOP4.1; no longer E40TOP4.1
- net AC7: now also F40BOT2.1; no longer E40BOT2.1
- net AC8: now also F40TOP12.1; no longer E40TOP12.1
- net AC9: now also F40BOT9.1; no longer E40BOT9.1
- net AND: now also D40BOT1.1; no longer F40BOT1.1
- net BREAK: now also D40BOT12.1; no longer F40BOT12.1
- net CA: now also D40BOT18.1; no longer F40BOT18.1
- net DCA: now also D40BOT4.1; no longer F40BOT4.1
- net DEFER: now also D40BOT16.1; no longer F40BOT15.1
- net EXECUTE: now also D40BOT15.1; no longer F40BOT16.1
- net FETCH: now also D40BOT14.1; no longer F40BOT14.1
- net GND: now also GND.1; no longer C40BOT13.1, D40BOT13.1, E40BOT13.1, F40BOT13.1, GND1-1.KL, GND1-2.KL, GND2-1.KL, GND2-2.KL, X3-1.KL, X3-2.KL, X4-1.KL, X4-2.KL
- net ION: now also D40BOT19.1; no longer F40BOT19.1
- net IOT: now also D40BOT9.1; no longer F40TOP13.1
- net ISZ: now also D40BOT3.1; no longer F40BOT3.1
- net JMP: now also D40BOT6.1; no longer F40BOT6.1
- net JMS: now also D40BOT5.1; no longer F40BOT5.1
- net MA0: now also E40TOP2.1; no longer D40TOP2.1
- net MA1: now also E40BOT4.1; no longer D40BOT4.1
- net MA10: now also F40TOP15.1; no longer E40TOP15.1
- net MA11: now also F40BOT18.1; no longer E40BOT18.1
- net MA2: now also E40TOP7.1; no longer D40TOP7.1
- net MA3: now also E40BOT12.1; no longer D40BOT12.1
- net MA4: now also E40TOP15.1; no longer D40TOP15.1
- net MA5: now also E40BOT18.1; no longer D40BOT18.1
- net MA6: now also F40TOP2.1; no longer E40TOP2.1
- net MA7: now also F40BOT4.1; no longer E40BOT4.1
- net MA8: now also F40TOP7.1; no longer E40TOP7.1
- net MA9: now also F40BOT12.1; no longer E40BOT12.1
- net MB0: now also E40TOP3.1; no longer D40TOP3.1
- net MB1: now also E40BOT3.1; no longer D40BOT3.1
- net MB10: now also F40TOP16.1; no longer E40TOP16.1
- net MB11: now also F40BOT17.1; no longer E40BOT17.1
- net MB2: now also E40TOP8.1; no longer D40TOP8.1
- net MB3: now also E40BOT11.1; no longer D40BOT11.1
- net MB4: now also E40TOP16.1; no longer D40TOP16.1
- net MB5: now also E40BOT17.1; no longer D40BOT17.1
- net MB6: now also F40TOP3.1; no longer E40TOP3.1
- net MB7: now also F40BOT3.1; no longer E40BOT3.1
- net MB8: now also F40TOP8.1; no longer E40TOP8.1
- net MB9: now also F40BOT11.1; no longer E40BOT11.1
- net MQ0: now also E40TOP5.1; no longer D40TOP5.1
- net MQ1: now also E40BOT1.1; no longer D40BOT1.1
- net MQ10: now also F40TOP18.1; no longer E40TOP18.1
- net MQ11: now also F40BOT15.1; no longer E40BOT15.1
- net MQ2: now also E40TOP13.1; no longer D40TOP13.1
- net MQ3: now also E40BOT6.1; no longer D40BOT6.1
- net MQ4: now also E40TOP18.1; no longer D40TOP18.1
- net MQ5: now also E40BOT15.1; no longer D40BOT15.1
- net MQ6: now also F40TOP5.1; no longer E40TOP5.1
- net MQ7: now also F40BOT1.1; no longer E40BOT1.1
- net MQ8: now also F40TOP13.1; no longer E40TOP13.1
- net MQ9: now also F40BOT6.1; no longer E40BOT6.1
- net OPR: now also D40BOT11.1; no longer F40BOT11.1
- net PAUSE: now also D40TOP17.1; no longer F40TOP17.1
- net PC0: now also E40TOP1.1; no longer D40TOP1.1
- net PC1: now also E40BOT5.1; no longer D40BOT5.1
- net PC10: now also F40TOP14.1; no longer E40TOP14.1
- net PC11: now also F40BOT19.1; no longer E40BOT19.1
- net PC2: now also E40TOP6.1; no longer D40TOP6.1
- net PC3: now also E40BOT14.1; no longer D40BOT14.1
- net PC4: now also E40TOP14.1; no longer D40TOP14.1
- net PC5: now also E40BOT19.1; no longer D40BOT19.1
- net PC6: now also F40TOP1.1; no longer E40TOP1.1
- net PC7: now also F40BOT5.1; no longer E40BOT5.1
- net PC8: now also F40TOP6.1; no longer E40TOP6.1
- net PC9: now also F40BOT14.1; no longer E40BOT14.1
- net RUN: now also D40TOP18.1; no longer F40TOP18.1
- net TAD: now also D40BOT2.1; no longer F40BOT2.1
- net WC: now also D40BOT17.1; no longer F40BOT17.1
Other:
- note added: "All bulbs are OL-1."
- note added: "Note: No common between logic GND and 15V GND!"
- note removed: "TODO: Connect up the ribbons!"
