File: projects/Stearns Tester/Stearns.sch (EAGLE design)
At the start: 63 parts, among them IC1 MCP23S17SP, IC2 MCP23S17SP, IC3 MCP23S17SP, IC4 MCP23S17SP, IC5 MCP23S17SP, IC6 74LS06N

Commit message: Finish fixing "no such part in library" stuff.
Parts:
- UUT: device switch:710X -> dec-con:710X
Changed lines of the file:
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@@
 <layer number="101" name="Patch_Top" color="7" fill="1" visible="yes" active="yes"/>
 <layer number="102" name="Vscore" color="7" fill="1" visible="yes" active="yes"/>
+<layer number="103" name="ATT_MISO" color="7" fill="1" visible="yes" active="yes"/>
 <layer number="104" name="Name" color="7" fill="1" visible="yes" active="yes"/>
+<layer number="105" name="Beschreib" color="7" fill="1" visible="yes" active="yes"/>
+<layer number="106" name="BGA-Top" color="7" fill="1" visible="yes" active="yes"/>
+<layer number="107" name="BD-Top" color="7" fill="1" visible="yes" active="yes"/>
+<layer number="108" name="centerline" color="7" fill="1" visible="yes" active="yes"/>
 <layer number="116" name="Patch_BOT" color="7" fill="1" visible="yes" active="yes"/>
 <layer number="121" name="_tsilk" color="7" fill="1" visible="yes" active="yes"/>
 <layer number="122" name="_bsilk" color="7" fill="1" visible="yes" active="yes"/>
+<layer number="131" name="prix" color="7" fill="1" visible="yes" active="yes"/>
+<layer number="132" name="test" color="7" fill="1" visible="yes" active="yes"/>
 <layer number="151" name="HeatSink" color="7" fill="1" visible="yes" active="yes"/>
 <layer number="200" name="200bmp" color="7" fill="1" visible="yes" active="yes"/>
@@
 <part name="V9" library="supply2" deviceset="VCC" device=""/>
 <part name="V10" library="supply2" deviceset="VDD" device=""/>
-<part name="UUT" library="switch" deviceset="710X" device=""/>
+<part name="UUT" library="dec-con" deviceset="710X" device=""/>
 <part name="V12" library="supply2" deviceset="VCC" device=""/>
 <part name="V13" library="supply2" deviceset="VPP" device=""/>

Commit message: Update board in an attempt to match Warren's wiring. Add ground planes and minor tweaks prior to ordering boards.
Parts:
- removed A, B: M916, dec-m:M916
- added DEC: W971, dec-m:W971
- added ECS: W971ECS, dec-m:W971ECS
- added EDAC: W971EDAC, dec-m:W971EDAC
- C1: value (none) -> 47uF
- C2, C3, C4, C5, C6, C7: value (none) -> .22uF
- renumbered LUT_PWR to UUT_PWR
Connections:
- removed net AC2J: AX2.6, IC1.GPB2
- removed net BC2J: BX2.6, IC3.GPA4
- net AA1J: now also IC1.GPB7; no longer IC1.GPA0
- net AA2J: now also IC1.GPA7; no longer IC1.GPB0
- net AB1J: now also IC1.GPB6; no longer IC1.GPA1
- net AB2J: now also IC1.GPA6; no longer IC1.GPB1
- net AC1J: now also IC1.GPB5; no longer IC1.GPA2
- net AD1J: now also IC1.GPB4; no longer IC1.GPA3
- net AD2J: now also IC1.GPA4; no longer IC1.GPB3
- net AE1J: now also IC1.GPB3; no longer IC1.GPA4
- net AE2J: now also IC1.GPA3; no longer IC1.GPB4
- net AF1J: now also IC1.GPB2; no longer IC1.GPA5
- net AF2J: now also IC1.GPA2; no longer IC1.GPB5
- net AH1J: now also IC1.GPB1; no longer IC1.GPA6
- net AH2J: now also IC1.GPA1; no longer IC1.GPB6
- net AJ1J: now also IC1.GPB0; no longer IC1.GPA7
- net AJ2J: now also IC1.GPA0; no longer IC1.GPB7
- net AK1J: now also IC2.GPB7; no longer IC2.GPA0
- net AK2J: now also IC2.GPA0; no longer IC2.GPB0
- net AL1J: now also IC2.GPB6; no longer IC2.GPA1
- net AL2J: now also IC2.GPA1; no longer IC2.GPB1
- net AM1J: now also IC2.GPB5; no longer IC2.GPA2
- net AM2J: now also IC2.GPA2; no longer IC2.GPB2
- net AN1J: now also IC2.GPB4; no longer IC2.GPA3
- net AN2J: now also IC2.GPA3; no longer IC2.GPB3
- net AP1J: now also IC2.GPB3; no longer IC2.GPA4
- net AP2J: now also IC2.GPA4; no longer IC2.GPB4
- net AR1J: now also IC2.GPB2; no longer IC2.GPA5
- net AR2J: now also IC2.GPA5; no longer IC2.GPB5
- net AS1J: now also IC2.GPB1; no longer IC2.GPA6
- net AS2J: now also IC2.GPA6; no longer IC2.GPB6
- net AT2J: now also IC2.GPA7; no longer IC2.GPB7
- net AU1J: now also IC3.GPB7; no longer IC3.GPB0
- net AV1J: now also IC3.GPB6; no longer IC3.GPB1
- net BA1J: now also IC3.GPB5; no longer IC3.GPB2
- net BB1J: now also IC3.GPB4; no longer IC3.GPB3
- net BC1J: now also IC3.GPB3; no longer IC3.GPB4
- net BD1J: now also IC3.GPB2; no longer IC3.GPB5
- net BE1J: now also IC3.GPB1; no longer IC3.GPB6
- net BF1J: now also IC3.GPB0; no longer IC3.GPB7
- net BH1J: now also IC4.GPB7; no longer IC4.GPA0
- net BH2J: now also IC4.GPA0; no longer IC4.GPB0
- net BJ1J: now also IC4.GPB6; no longer IC4.GPA1
- net BJ2J: now also IC4.GPA1; no longer IC4.GPB1
- net BK1J: now also IC4.GPB5; no longer IC4.GPA2
- net BK2J: now also IC4.GPA2; no longer IC4.GPB2
- net BL1J: now also IC4.GPB4; no longer IC4.GPA3
- net BL2J: now also IC4.GPA3; no longer IC4.GPB3
- net BM1J: now also IC4.GPB3; no longer IC4.GPA4
- net BM2J: now also IC4.GPA4; no longer IC4.GPB4
- net BN1J: now also IC4.GPB2; no longer IC4.GPA5
- net BN2J: now also IC4.GPA5; no longer IC4.GPB5
- net BP1J: now also IC4.GPB1; no longer IC4.GPA6
- net BP2J: now also IC4.GPA6; no longer IC4.GPB6
- net BR1J: now also IC4.GPB0; no longer IC4.GPA7
- net BR2J: now also IC4.GPA7; no longer IC4.GPB7
- net BS1J: now also IC5.GPB7; no longer IC5.GPA0
- net BS2J: now also IC5.GPA0; no longer IC5.GPA4
- net BT2J: now also IC5.GPA1; no longer IC5.GPA5
- net BU1J: now also IC5.GPB5; no longer IC5.GPA2
- net BU2J: now also IC5.GPA2; no longer IC5.GPA6
- net BV1J: now also IC5.GPB4; no longer IC5.GPA3
- net BV2J: now also IC5.GPA3; no longer IC5.GPA7
- net GND: now also AX2.6, BX2.6, IC1.GPA5, IC2.GPB0, IC3.GPA4, IC5.GPB6; no longer IC2.GPA7, IC5.GPA1
- net N$1: now also DECAA1.P$2, ECSAA1.P$2, EDACAA1.P$2; no longer AA1.P$2
- net N$10: now also DECAL1.P$2, ECSAL1.P$2, EDACAL1.P$2; no longer AL1.P$2
- net N$11: now also DECAK1.P$2, ECSAK1.P$2, EDACAK1.P$2; no longer AK1.P$2
- net N$12: now also DECAJ1.P$2, ECSAJ1.P$2, EDACAJ1.P$2; no longer AJ1.P$2
- net N$13: now also DECAH1.P$2, ECSAH1.P$2, EDACAH1.P$2; no longer AH1.P$2
- net N$14: now also DECAF1.P$2, ECSAF1.P$2, EDACAF1.P$2; no longer AF1.P$2
- net N$15: now also DECAE1.P$2, ECSAE1.P$2, EDACAE1.P$2; no longer AE1.P$2
- net N$16: now also DECAD1.P$2, ECSAD1.P$2, EDACAD1.P$2; no longer AD1.P$2
- net N$17: now also DECAC1.P$2, ECSAC1.P$2, EDACAC1.P$2; no longer AC1.P$2
- net N$18: now also DECAB1.P$2, ECSAB1.P$2, EDACAB1.P$2; no longer AB1.P$2
- net N$19: now also DECAA2.P$2, ECSAA2.P$2, EDACAA2.P$2; no longer AA2.P$2
- net N$2: now also DECAV1.P$2, ECSAV1.P$2, EDACAV1.P$2; no longer AV1.P$2
- net N$20: now also DECAB2.P$2, ECSAB2.P$2, EDACAB2.P$2; no longer AB2.P$2
- net N$21: now also DECAC2.P$2, ECSAC2.P$2, EDACAC2.P$2; no longer AC2.P$2
- net N$22: now also DECAD2.P$2, ECSAD2.P$2, EDACAD2.P$2; no longer AD2.P$2
- net N$23: now also DECAE2.P$2, ECSAE2.P$2, EDACAE2.P$2; no longer AE2.P$2
- net N$24: now also DECAF2.P$2, ECSAF2.P$2, EDACAF2.P$2; no longer AF2.P$2
- net N$25: now also DECAH2.P$2, ECSAH2.P$2, EDACAH2.P$2; no longer AH2.P$2
- net N$26: now also DECAJ2.P$2, ECSAJ2.P$2, EDACAJ2.P$2; no longer AJ2.P$2
- net N$27: now also DECAK2.P$2, ECSAK2.P$2, EDACAK2.P$2; no longer AK2.P$2
- net N$28: now also DECAL2.P$2, ECSAL2.P$2, EDACAL2.P$2; no longer AL2.P$2
- net N$29: now also DECAM2.P$2, ECSAM2.P$2, EDACAM2.P$2; no longer AM2.P$2
- net N$3: now also DECAU1.P$2, ECSAU1.P$2, EDACAU1.P$2; no longer AU1.P$2
- net N$30: now also DECAN2.P$2, ECSAN2.P$2, EDACAN2.P$2; no longer AN2.P$2
- net N$31: now also DECAP2.P$2, ECSAP2.P$2, EDACAP2.P$2; no longer AP2.P$2
- net N$32: now also DECAR2.P$2, ECSAR2.P$2, EDACAR2.P$2; no longer AR2.P$2
- net N$33: now also DECAS2.P$2, ECSAS2.P$2, EDACAS2.P$2; no longer AS2.P$2
- net N$34: now also DECAT2.P$2, ECSAT2.P$2, EDACAT2.P$2; no longer AT2.P$2
- net N$35: now also DECAU2.P$2, ECSAU2.P$2, EDACAU2.P$2; no longer AU2.P$2
- net N$36: now also DECAV2.P$2, ECSAV2.P$2, EDACAV2.P$2; no longer AV2.P$2
- net N$37: now also DECBA2.P$2, ECSBA2.P$2, EDACBA2.P$2; no longer BA2.P$2
- net N$38: now also DECBB2.P$2, ECSBB2.P$2, EDACBB2.P$2; no longer BB2.P$2
- net N$39: now also DECBC2.P$2, ECSBC2.P$2, EDACBC2.P$2; no longer BC2.P$2
- net N$4: now also DECAT1.P$2, ECSAT1.P$2, EDACAT1.P$2; no longer AT1.P$2
- net N$40: now also DECBD2.P$2, ECSBD2.P$2, EDACBD2.P$2; no longer BD2.P$2
- net N$41: now also DECBE2.P$2, ECSBE2.P$2, EDACBE2.P$2; no longer BE2.P$2
- net N$42: now also DECBF2.P$2, ECSBF2.P$2, EDACBF2.P$2; no longer BF2.P$2
- net N$43: now also DECBH2.P$2, ECSBH2.P$2, EDACBH2.P$2; no longer BH2.P$2
- net N$44: now also DECBJ2.P$2, ECSBJ2.P$2, EDACBJ2.P$2; no longer BJ2.P$2
- net N$45: now also DECBK2.P$2, ECSBK2.P$2, EDACBK2.P$2; no longer BK2.P$2
- net N$46: now also DECBL2.P$2, ECSBL2.P$2, EDACBL2.P$2; no longer BL2.P$2
- net N$47: now also DECBM2.P$2, ECSBM2.P$2, EDACBM2.P$2; no longer BM2.P$2
- net N$48: now also DECBN2.P$2, ECSBN2.P$2, EDACBN2.P$2; no longer BN2.P$2
- net N$49: now also DECBP2.P$2, ECSBP2.P$2, EDACBP2.P$2; no longer BP2.P$2
- net N$5: now also DECAS1.P$2, ECSAS1.P$2, EDACAS1.P$2; no longer AS1.P$2
- net N$50: now also DECBR2.P$2, ECSBR2.P$2, EDACBR2.P$2; no longer BR2.P$2
- net N$51: now also DECBS2.P$2, ECSBS2.P$2, EDACBS2.P$2; no longer BS2.P$2
- net N$52: now also DECBT2.P$2, ECSBT2.P$2, EDACBT2.P$2; no longer BT2.P$2
- net N$53: now also DECBU2.P$2, ECSBU2.P$2, EDACBU2.P$2; no longer BU2.P$2
- net N$54: now also DECBV2.P$2, ECSBV2.P$2, EDACBV2.P$2; no longer BV2.P$2
- net N$55: now also DECBA1.P$2, ECSBA1.P$2, EDACBA1.P$2; no longer BA1.P$2
- net N$56: now also DECBB1.P$2, ECSBB1.P$2, EDACBB1.P$2; no longer BB1.P$2
- net N$57: now also DECBC1.P$2, ECSBC1.P$2, EDACBC1.P$2; no longer BC1.P$2
- net N$58: now also DECBD1.P$2, ECSBD1.P$2, EDACBD1.P$2; no longer BD1.P$2
- net N$59: now also DECBE1.P$2, ECSBE1.P$2, EDACBE1.P$2; no longer BE1.P$2
- net N$6: now also DECAR1.P$2, ECSAR1.P$2, EDACAR1.P$2; no longer AR1.P$2
- net N$60: now also DECBF1.P$2, ECSBF1.P$2, EDACBF1.P$2; no longer BF1.P$2
- net N$61: now also DECBH1.P$2, ECSBH1.P$2, EDACBH1.P$2; no longer BH1.P$2
- net N$62: now also DECBJ1.P$2, ECSBJ1.P$2, EDACBJ1.P$2; no longer BJ1.P$2
- net N$63: now also DECBK1.P$2, ECSBK1.P$2, EDACBK1.P$2; no longer BK1.P$2
- net N$64: now also DECBL1.P$2, ECSBL1.P$2, EDACBL1.P$2; no longer BL1.P$2
- net N$65: now also DECBM1.P$2, ECSBM1.P$2, EDACBM1.P$2; no longer BM1.P$2
- net N$66: now also DECBN1.P$2, ECSBN1.P$2, EDACBN1.P$2; no longer BN1.P$2
- net N$67: now also DECBP1.P$2, ECSBP1.P$2, EDACBP1.P$2; no longer BP1.P$2
- net N$68: now also DECBR1.P$2, ECSBR1.P$2, EDACBR1.P$2; no longer BR1.P$2
- net N$69: now also DECBS1.P$2, ECSBS1.P$2, EDACBS1.P$2; no longer BS1.P$2
- net N$7: now also DECAP1.P$2, ECSAP1.P$2, EDACAP1.P$2; no longer AP1.P$2
- net N$70: now also DECBT1.P$2, ECSBT1.P$2, EDACBT1.P$2; no longer BT1.P$2
- net N$71: now also DECBU1.P$2, ECSBU1.P$2, EDACBU1.P$2; no longer BU1.P$2
- net N$72: now also DECBV1.P$2, ECSBV1.P$2, EDACBV1.P$2; no longer BV1.P$2
- net N$8: now also DECAN1.P$2, ECSAN1.P$2, EDACAN1.P$2; no longer AN1.P$2
- net N$9: now also DECAM1.P$2, ECSAM1.P$2, EDACAM1.P$2; no longer AM1.P$2
- net PROBE1: now also IC5.GPA4; no longer IC5.GPB4
- net PROBE2: now also IC5.GPA5; no longer IC5.GPB5
- net PROBE3: now also IC5.GPA6; no longer IC5.GPB6
- net PROBE4: now also IC5.GPA7; no longer IC5.GPB7
- net VPP: now also IC3.GPA2
Other:
- moved on the sheet: R1
