File: projects/DEC/Mxxx/M8341/M8341D.sch (EAGLE design)
At the start: 101 parts

Commit message: Bring M8341 CUPL and Verilog up to date.
Connections:
- net N$10 renamed TP
Changed lines of the file:
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@@
 </segment>
 </net>
-<net name="N$10" class="0">
+<net name="TP" class="0">
 <segment>
 <pinref part="E2" gate="B" pin="I0"/>
