File: projects/DEC/Mxxx/M8650/M8650D.brd (EAGLE design)
At the start: 265.3 x 214.6 mm, 193 parts, among them Q1 2N3009B, Q2 MPS6534, Q3 MPS6534D, T1 16-0951, Y1 19.661 MHz

Commit message: Add 1013 UART to dec-con.lbr. Fix "no such part in library" stuff for DEC subtree.
Connections:
- net 3.3V renamed +3V3
Routing:
- net +3V3: track 972.2 -> 973.9 mm

Commit message: Fix a problem in the M8650 drawings where BTP3 and !TP3 names were swapped.
Connections:
- net !TP3: now also E42.4, E45.3, E47.5, E47.9; no longer E25.2, E34.14, E41.13, E42.3, E44.13
- net BTP3: now also E25.2, E34.14, E41.13, E42.3, E44.13; no longer E42.4, E45.3, E47.5, E47.9
Routing:
- net BTP3: track 86.5 -> 255.5 mm
- net !TP3: track 255.5 -> 86.5 mm
Changed lines of the file:
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@@
 <wire x1="10.16" y1="76.2" x2="10.16" y2="78.74" width="0.4064" layer="1"/>
 </signal>
-<signal name="!TP3">
+<signal name="BTP3">
 <contactref element="E34" pad="14"/>
 <contactref element="E42" pad="3"/>
@@
 <via x="52.07" y="129.54" extent="1-16" drill="0.8128"/>
 </signal>
-<signal name="BTP3">
+<signal name="!TP3">
 <contactref element="E42" pad="4"/>
 <contactref element="E47" pad="5"/>
