File: projects/DEC/Mxxx/M8650/M8650D+cpld+.brd (EAGLE design)
At the start: 265.3 x 214.6 mm, 127 parts, among them IC1 74S138N, IC12 74LS27N, IC2 74S138N, IC3 74151N, IC4 74151N, IC5 74S138N, IC6 74S138N, IC7 74S138N, IC8 74151N, IC9 74S11N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

Commit message: Update snapshot of M8650 PLD effort.
Parts:
- removed E17: 7493N, 74xx-us:DIL14
- added IC10: 74LS08N, 74xx-us:DIL14
- OSC, OSC1: value 19.6608 MHz -> 3.6864 MHz
- moved C9 1.27 mm to (215.9, 26.7)
Connections:
- removed net BD153600: E17.8, IC8.12
- removed net BD307200: E17.9
- removed net BD614400: E17.1, E17.12
- removed net BD76800: E17.11, E18.14, IC8.13
- removed net CLK: E17.14, OSC.5, OSC1.8
- new net BD115200: E18.1, E18.12, IC8.13
- new net BD230400: E18.14, IC8.12, OSC.5, OSC1.8
- new net BD57600: E18.9, IC9.3, IC9.4
- new net N$3: E18.2, E18.3, IC9.6
- new net TP_AB1: IC10.3, U$2.AB1
- new net TP_BA1: IC10.6, U$2.BA1
- new net TP_BB1: IC10.8, U$2.BB1
- new net TP_CA1: IC10.11, U$2.CA1
- net BD38400: now also E18.8, IC9.5; no longer E18.12
- net DOTPC: now also IC10.10, IC10.9
- net GND: now also IC10.7; no longer E17.10, E17.2, E17.3, E18.1, E18.2, E18.3
- net N$103: no longer E25.5
- net RX_ACTIVE: now also IC10.1, IC10.2
- net TP3: now also IC10.12, IC10.13
- net TX_ACTIVE: now also E25.5, IC10.4, IC10.5
- net VCC: now also IC10.14; no longer E17.5
Routing:
- net MD08_L: track 220.0 -> 11.2 mm, vias 2 -> 1
- net GND: track 2706.5 -> 2727.9 mm, vias 11 -> 12
- net N$103: track 73.6 -> 71.8 mm
- net TX_ACTIVE: track 281.0 -> 281.6 mm
