File: projects/DEC/BM8L/BM8L.sch (EAGLE design)
At the start: 66 parts

Commit message: Don't use "INT" and "RETURN" as signal names (added trailing H).
Connections:
- net INT renamed INTH
- net RETURN renamed RETURNH
Changed lines of the file:
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@@
 </segment>
 </net>
-<net name="RETURN" class="0">
+<net name="RETURNH" class="0">
 <segment>
 <pinref part="C08" gate="E1" pin="OUT"/>
@@
 </segment>
 </net>
-<net name="INT" class="0">
+<net name="INTH" class="0">
 <segment>
 <pinref part="D12" gate="E1" pin="1"/>
@@
 </segment>
 </net>
-<net name="RETURN" class="0">
+<net name="RETURNH" class="0">
 <segment>
 <pinref part="AB07" gate="AR2" pin="P$2"/>
